File: sasquatch_v2.sch (EAGLE design)
At the start: 54 parts, among them M1 40V, M2 40V, U1 BLE112-A, U2 LM22677TJ-5.0/NOPB, U3 LM3150MH/NOPB

Commit message: Added WEBENCH Buildit Boards
Parts:
- removed C1: 22uF, SparkFun-Capacitors:22UF-16V-20%-(1210)
- removed C2: 2.2uF, SparkFun-Capacitors:2.2UF-10V-20%(0603)
- removed C3: (no value), SparkFun-Capacitors:CAP0402-CAP
- removed C6: 4.7uF, SparkFun-Capacitors:4.7UF-6.3V-10%(0603)0603
- removed D1: MBRS140, diode:SCHOTTKY-DIODESMD
- removed GND10, GND11, GND4, GND5, GND6, GND7, GND8, GND9, GND_1: WB_GND, AcceleratedDesigns_Lib:WB_GNDWB_GND
- removed L1: B82477G2103M, senior_design_library:B82477G2103M
- removed R8: 300R, SparkFun-Resistors:RESISTOR0603
- removed R9: 18k2, SparkFun-Resistors:RESISTOR0603
- removed U$2: LT3514, senior_design_library:LT3514
- removed U$5: FQB33N10TM, senior_design_library:FQB33N10TM
- added F1, F2: PTCPTH, SparkFun-PowerIC:PTCPTH
- added J$4: CON-POWERPOLE, con-powerpole:CON-POWERPOLE
- added T$1: FQB33N10TM, senior_design_library:FQB33N10TM
- U$1: value MAX1607 -> STMPS2141MTR; device senior_design_library:MAX1607 -> senior_design_library:STMPS2141MTR
Connections:
- removed net 11: CBYP_1.1@1, CIN_4.+@1, M1.DRAIN@1, M1.DRAIN@2, M1.DRAIN@3, M1.DRAIN@4, RON_1.1@1, U3.VIN@2
- removed net 2: CINX_1.1@1, CIN_1.+@1, CIN_2.+@1, CIN_3.+@1, U2.VIN@1
- removed net N$13: GND10.1@1, RFB3.2@2
- removed net N$3: R9.2, U$2.RT
- removed net N$4: C2.2, U$2.SKY
- removed net N$5: C3.2, U$2.RUN/SS1, U$2.RUN/SS3, U$2.RUN/SS4
- removed net N$6: R8.2, U$2.PG
- removed net N$7: D1.A, U$2.DA1
- removed net N$8: D1.C, U$2.SW1
- new net BAT_GND: J$4.-, T$1.D
- new net VIN: CBYP_1.1@1, CINX_1.1@1, CIN_4.+@1, J$4.+, M1.DRAIN@1, M1.DRAIN@2, M1.DRAIN@3, M1.DRAIN@4, RON_1.1@1, T$1.G, U2.VIN@1
- net 0: no longer GND_1.1@1
- net 12: no longer COUT_2.-@2, CSS_1.2@2, CVCC_1.2@2, GND11.1@1, GND4.1@1, GND5.1@1, GND6.1@1, GND7.1@1, GND8.1@1, GND9.1@1, M2.SOURCE@6, M2.SOURCE@7, M2.SOURCE@8, U3.DAP@14, U3.PGND@15, U3.SGND@5, U3.SGND@9
- net GND: now also COUT_2.-@2, CSS_1.2@2, M2.SOURCE@6, M2.SOURCE@7, M2.SOURCE@8, RFB3.2@2, T$1.S, U3.DAP@14, U3.PGND@15, U3.SGND@5, U3.SGND@9; no longer C1.1, C3.1, C6.1, U$1.GND
- net N$1: now also CIN_1.+@1, CIN_2.+@1, CIN_3.+@1; no longer C1.2, C2.1, C6.2, L1.1, U$2.EN/UVLO, U$2.VIN
- net N$2: now also U3.VIN@2; no longer L1.2, U$2.SW5
Other:
- moved on the sheet: CBST_1, CBST_2, CBYP_1, CFF_1, CINX_1, CIN_1, CIN_2, CIN_3, CIN_4, COUT_1, COUT_2, CSS_1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
